File: wled_2_digi/wled_2_digi.kicad_pcb (KiCad board)
At the start: 2 copper layers, 75 x 38 mm, 31 parts, among them J1 Barrel_Jack_Switch, J3 Screw_Terminal_01x04, J4 Screw_Terminal_01x04, Q2 AP15P04S, Q3 MMBT2222A, Q4 MMBT2222A, Q5 AP15P04S, U1 74AHCT125, U2 AP63205WU, U3 Screw Terminal

Commit message: Add QR Code
Parts:
- added G***: LOGO, LOGO, B.Cu at (103.7, 77.9)
Other:
- board text added: "DerNiccoo wled_2_digi"

Commit message: Moved components closer
Parts:
- moved C4 3.87 mm to (118.4, 76.2)
- moved U1 3.87 mm to (123.5, 73.0)
Routing:
- net HS_Enabled_2: track 45.4 -> 37.1 mm
- net Net-(R5-Pad1): track 22.5 -> 15.6 mm
- net Net-(R8-Pad1): track 33.3 -> 26.8 mm
- net Net-(R4-Pad1): track 25.5 -> 19.2 mm
- net GND: track 23.2 -> 18.6 mm
- net Net-(R9-Pad1): track 30.9 -> 26.8 mm
- net +5V: track 41.9 -> 38.1 mm
- net DATA2: track 12.2 -> 14.4 mm
- net DATA1: track 17.8 -> 20.0 mm
- net CLK1: track 21.8 -> 20.3 mm
- net CLK2: track 22.5 -> 23.1 mm
Other:
- board text added: "DerNiccoo wled_2_digi v1"
- board text removed: "DerNiccoo wled_2_digi"
