File: wled_esp_board/wled_esp_board.kicad_sch (KiCad schematic)
At the start: 26 parts, among them J1 Conn_01x09_Pin, J2 USB_C_Receptacle_USB2.0_16P, J3 Conn_01x09_Pin, J4 Conn_01x09_Pin, J5 Conn_01x09_Pin, SW1 Reset, SW2 Boot, U1 ESP32-S3-WROOM-1, U2 USBLC6-2SC6, U3 AP63203WU

Commit message: Update QR Code on base board
Parts:
- added J10, J6, J7, J8, J9: Conn_01x01_Pin, Connector_PinHeader_1.00mm:PinHeader_1x01_P1.00mm_Horizontal, symbol Connector:Conn_01x01_Pin
Connections:
- net GND: now also J10.1 (Pin_1), J6.1 (Pin_1), J7.1 (Pin_1), J8.1 (Pin_1), J9.1 (Pin_1)
